File: hw/2x5pin_2.54mm_pitch/tpm_2x5pin.kicad_pcb (KiCad board)
At the start: 2 copper layers, 24.9 x 16.8 mm, 11 parts, among them J1 Conn_02x05_Odd_Even, U1 SLB9665

Commit message: Add UserComments layer with board setup and characteristics
Signed-off-by: Michał Żygowski <michal.zygowski@3mdeb.com>
Other:
- board text added: "0"
- board text added: "0 mm"
- board text added: "0.01 mm"
- board text added: "0.02"
- board text added: "0.035 mm"
- board text added: "0.2000 mm / 0.1270 mm"
- board text added: "0.3000 mm"
- board text added: "1"
- board text added: "1.51 mm"
- board text added: "1.6000 mm"
- board text added: "2"
- board text added: "24.8920 mm x 16.7767 mm"
- board text added: "3.3"
- board text added: "4.5"
- board text added: "B.Cu"
- board text added: "B.Mask"
- board text added: "B.Paste"
- board text added: "B.Silkscreen"
- board text added: "BOARD CHARACTERISTICS"
- board text added: "Board Thickness:"
- board text added: "Board overall dimensions:"
- board text added: "Bottom Silk Screen"
- board text added: "Bottom Solder Mask"
- board text added: "Bottom Solder Paste"
- board text added: "Castellated pads:"
- board text added: "Color"
- board text added: "Copper Finish:"
- board text added: "Copper Layer Count:"
- board text added: "Dielectric 1"
- board text added: "ENIG"
- board text added: "Edge card connectors:"
- board text added: "Epoxy"
- board text added: "Epsilon R"
- board text added: "F.Cu"
- board text added: "F.Mask"
- board text added: "F.Paste"
- board text added: "F.Silkscreen"
- board text added: "FR4"
- board text added: "FR4 natural"
- board text added: "Green"
- board text added: "Impedance Control:"
- board text added: "Layer Name"
- board text added: "Liquid Photo"
- board text added: "Loss Tangent"
- board text added: "Material"
- board text added: "Min hole diameter:"
- board text added: "Min track/spacing:"
- board text added: "No"
- board text added: "Plated Board Edge:"
- board text added: "Thickness (mm)"
- board text added: "Top Silk Screen"
- board text added: "Top Solder Mask"
- board text added: "Top Solder Paste"
- board text added: "Type"
- board text added: "White"
- board text added: "copper"
- board text added: "core"
