File: hw/2x5pin_2.54mm_pitch/tpm_2x5pin.kicad_sch (KiCad schematic)
At the start: 9 parts, among them J1 Conn_02x05_Odd_Even, U1 SLB9665

Commit message: Add UserComments layer with board setup and characteristics
Signed-off-by: Michał Żygowski <michal.zygowski@3mdeb.com>
Parts:
- J1: Supplier and ref (none) -> https://www.mouser.pl/ProductDetail/Samtec/SSQ-105-01-L-D?q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
- U1: Supplier and ref (none) -> https://www.mouser.pl/ProductDetail/Infineon-Technologies/S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
Changed lines of the file:
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@@
+      (effects (font (size 1.27 1.27)) hide)
+    )
+    (property "Supplier and ref" "https://www.mouser.pl/ProductDetail/Infineon-Technologies/SLB9665TT20FW563XUMA3?qs=gZXFycFWdAOgz%2FB%2Fifoq1g%3D%3D" (at 248.92 139.7 0)
       (effects (font (size 1.27 1.27)) hide)
     )
@@
       (effects (font (size 1.27 1.27)) hide)
     )
+    (property "Supplier and ref" "https://www.mouser.pl/ProductDetail/Samtec/SSQ-105-01-L-D?qs=%252BZP6%2F%252BtExtBCTa%252BcdSc7DA%3D%3D" (at 186.69 148.59 0)
+      (effects (font (size 1.27 1.27)) hide)
+    )
